File: pcb/teds-business-card/teds-business-card.kicad_sch (KiCad schematic)
At the start: 5 parts, among them U1 NT3H2111W0FHKH

Commit message: add prod files
Parts:
- C1: footprint Capacitor_SMD:C_0201_0603Metric -> easyeda2kicad:C0603
Changed lines of the file:
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@@
 			)
 		)
-		(property "Footprint" "Capacitor_SMD:C_0201_0603Metric"
+		(property "Footprint" "easyeda2kicad:C0603"
 			(at 87.63 98.0948 0)
 			(effects
